Commit message: 02/04/25 - added filter to smooth q7 values in main.py

File: src/path_planning/data/models/base/model.urdf (robot description, URDF)
Before this commit: robot base, 1 links, 0 joints
Links:
- link base: geometry collision box size=0.4 0.2 0.2; visual box size=0.4 0.2 0.2

File: src/path_planning/data/models/brick/model.urdf (robot description, URDF)
Before this commit: robot brick, 1 links, 0 joints
Links:
- link brick: geometry collision box size=0.04 0.08 0.04; visual box size=0.04 0.08 0.04
